File: mcu.kicad_sch (KiCad schematic)
At the start: 0 parts

Commit message: added 5v power supplies, 12v LDO, connectors, etc.
Parts:
- added C1, C2, C3, C4: 22pF, Capacitor_SMD:C_0805_2012Metric_Pad1.18x1.45mm_HandSolder, symbol Device:C
- added R1: 1M, Resistor_SMD:R_0805_2012Metric_Pad1.20x1.40mm_HandSolder, symbol Device:R_US
- added R2: 10K, Resistor_SMD:R_0805_2012Metric_Pad1.20x1.40mm_HandSolder, symbol Device:R_US
- added U2: ATmega328P-A, Package_QFP:TQFP-32_7x7mm_P0.8mm, symbol MCU_Microchip_ATmega:ATmega328P-A
- added Y1: Crystal, symbol Device:Crystal
Connections:
- new net +5V: C3.1, C4.2, R2.1, U2.18 (AVCC), U2.4 (VCC), U2.6 (VCC)
- new net EN1: U2.23 (PC0)
- new net EN2: U2.24 (PC1)
- new net EN3: U2.25 (PC2)
- new net EN4: U2.26 (PC3)
- new net EN5: U2.27 (PC4)
- new net GND: C1.2, C2.2, C3.2, C4.1, U2.21 (GND), U2.3 (GND), U2.5 (GND)
- new net MISO: U2.16 (PB4)
- new net MOSI: U2.15 (PB3)
- new net RESET: R2.2, U2.29 (~{RESET}/PC6)
- new net RX_IN: U2.30 (PD0)
- new net SCK: U2.17 (PB5)
- new net TX_OUT: U2.31 (PD1)
- new net XTAL1: C1.1, R1.1, U2.7 (XTAL1/PB6), Y1.1
- new net XTAL2: C2.1, R1.2, U2.8 (XTAL2/PB7), Y1.2
